File: board/MacroPad.brd (EAGLE design)
At the start: 129.5 x 77.1 mm, 70 parts, among them IC1 MIC5219BM5, J1 USB4085-GF-A_REVA4, U1 ATMEGA32U4-AUR, Y1 XRCGB16M000FXN00R0

Commit message: Added CS pin for display to schematic + board
The CS pin was initially left not connected intentionally, because I was led to believe that the CS pin was only needed when using multiple devices on SPI. However, for displays like the one used, the CS pin is needed for proper display initialization. DO NOT use earlier schematics and/or board files, as these do not have a properly working display connector.
Connections:
- removed net N$24: DS1.7
- new net D9: DS1.7, U1.29
Routing:
- net D9: track 0.00 -> 41.4 mm, vias 0 -> 2
Changed lines of the file:
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@@
 <drawing>
 <settings>
-<setting alwaysvectorfont="yes"/>
+<setting alwaysvectorfont="no"/>
 <setting verticaltext="up"/>
 </settings>
@@
 <wire x1="116.078" y1="62.484" x2="115.062" y2="63.5" width="0.254" layer="1"/>
 <wire x1="116.078" y1="58.42" x2="116.078" y2="62.484" width="0.254" layer="1"/>
-<wire x1="117.856" y1="56.642" x2="116.078" y2="58.42" width="0.254" layer="1"/>
+<wire x1="117.856" y1="56.642" x2="116.459" y2="58.039" width="0.254" layer="1"/>
+<wire x1="116.459" y1="58.039" x2="116.078" y2="58.42" width="0.254" layer="1"/>
 <wire x1="117.856" y1="37.084" x2="117.856" y2="56.642" width="0.254" layer="1"/>
 <wire x1="106.68" y1="25.908" x2="117.856" y2="37.084" width="0.254" layer="1"/>
@@
 <via x="111.76" y="34.29" extent="1-16" drill="0.35"/>
 </signal>
-<signal name="N$24">
+<signal name="D9">
 <contactref element="DS1" pad="7"/>
+<contactref element="U1" pad="29"/>
+<via x="115.189" y="61.722" extent="1-16" drill="0.35"/>
+<wire x1="113.63" y1="61.76" x2="115.151" y2="61.76" width="0.254" layer="1"/>
+<wire x1="115.151" y1="61.76" x2="115.189" y2="61.722" width="0.254" layer="1"/>
+<wire x1="115.189" y1="61.722" x2="115.189" y2="55.686225" width="0.254" layer="16"/>
+<wire x1="115.189" y1="55.686225" x2="114.7346" y2="55.231825" width="0.254" layer="16"/>
+<wire x1="114.7346" y1="34.7246" x2="113.03" y2="33.02" width="0.254" layer="16"/>
+<wire x1="114.7346" y1="55.231825" x2="114.7346" y2="34.7246" width="0.254" layer="16"/>
+<via x="111.76" y="33.02" extent="1-16" drill="0.35"/>
+<wire x1="113.03" y1="33.02" x2="111.76" y2="33.02" width="0.254" layer="16"/>
+<wire x1="111.76" y1="33.02" x2="110.998" y2="32.258" width="0.254" layer="1"/>
+<wire x1="110.998" y1="32.258" x2="108.501575" y2="32.258" width="0.254" layer="1"/>
+<wire x1="105.943575" y1="29.7" x2="104.14" y2="29.7" width="0.254" layer="1"/>
+<wire x1="108.501575" y1="32.258" x2="105.943575" y2="29.7" width="0.254" layer="1"/>
 </signal>
 <signal name="D15">
